Commit message: added ros camera

File: elfin/elfin_description/urdf/elfin3.urdf.xacro (robot description, xacro)
@@ -5,4 +5,5 @@
   <xacro:include filename="$(find elfin_description)/urdf/elfin_transmission.xacro" />
   <xacro:property name="PI" value="3.1415926535897931"/>
+  <xacro:property name="camera_link" value="0.05" /> <!-- Size of square 'camera' box -->
   <link name="world"/>
   <joint name="world_base" type="fixed">
@@ -430,3 +431,30 @@
       link="elfin_dummy_gripper" />
   </joint>
+   <joint name="camera_joint" type="fixed">
+      <axis xyz="0 1 0" />
+      <origin xyz="${camera_link} 0 0" rpy="0 0 0"/>
+      <parent link="elfin_dummy_gripper"/>
+      <child link="camera_link"/>
+    </joint>
+    <!-- Camera -->
+    <link name="camera_link">
+      <collision>
+        <origin xyz="0 0 0" rpy="0 0 0"/>
+        <geometry>
+      <box size="${camera_link} ${camera_link} ${camera_link}"/>
+        </geometry>
+      </collision>
+      <visual>
+        <origin xyz="0 0 0" rpy="0 0 0"/>
+        <geometry>
+      <box size="${camera_link} ${camera_link} ${camera_link}"/>
+        </geometry>
+        <material name="red"/>
+      </visual>
+      <inertial>
+        <mass value="1e-5" />
+        <origin xyz="0 0 0" rpy="0 0 0"/>
+        <inertia ixx="1e-6" ixy="0" ixz="0" iyy="1e-6" iyz="0" izz="1e-6" />
+      </inertial>
+    </link>
 </robot>
