Commit message: fixed camera orientation

File: elfin/elfin_description/urdf/elfin3.urdf_visualservo.xacro (robot description, xacro)
@@ -411,18 +411,18 @@
       velocity="1.57" />
   </joint>
-  <link name="elfin_dummy_gripper"/>
-  <joint name="elfin_dummy_joint" type="fixed">
-    <origin
-      xyz="0 -0.111 0"
+  <link name="elfin_end_link"/>
+  <joint name="elfin_end_joint" type="fixed">
+    <origin
+      xyz="0 -0.091 0"
       rpy="${PI/2} ${-PI/2} 0" />
     <parent
       link="elfin_link6" />
     <child
-      link="elfin_dummy_gripper" />
+      link="elfin_end_link" />
   </joint>
   <joint name="camera_joint" type="fixed">
     <axis xyz="0 1 0" />
-    <origin xyz="${camera_link} 0 0" rpy="0 0 0"/>
-    <parent link="elfin_dummy_gripper"/>
+    <origin xyz="0 0 0" rpy="0 ${-PI/2} 0"/>
+    <parent link="elfin_end_link"/>
     <child link="camera_link"/>
   </joint>

Commit message: updated frames

File: elfin/elfin_description/urdf/elfin3.urdf_visualservo.xacro (robot description, xacro)
@@ -422,5 +422,5 @@
   </joint>
   <joint name="camera_joint" type="fixed">
-    <axis xyz="0 1 0" />
+    <axis xyz="0 1 1" />
     <origin xyz="0 0 0" rpy="0 ${-PI/2} 0"/>
     <parent link="elfin_end_link"/>

Commit message: updated aruco to use other package

File: elfin/elfin_description/urdf/elfin3.urdf_visualservo.xacro (robot description, xacro)
@@ -422,5 +422,5 @@
   </joint>
   <joint name="camera_joint" type="fixed">
-    <axis xyz="0 1 1" />
+    <axis xyz="0 0 0" />
     <origin xyz="0 0 0" rpy="0 ${-PI/2} 0"/>
     <parent link="elfin_end_link"/>

Commit message: updated markers

File: elfin/elfin_description/urdf/elfin3.urdf_visualservo.xacro (robot description, xacro)
@@ -423,6 +423,6 @@
   <joint name="camera_joint" type="fixed">
     <axis xyz="0 0 0" />
-    <origin xyz="0 0 0" rpy="0 ${-PI/2} 0"/>
-    <parent link="elfin_end_link"/>
+    <origin xyz="0 -0.079 0" rpy="${PI} 0 -${PI/2}"/>
+    <parent link="elfin_link6"/>
     <child link="camera_link"/>
   </joint>
@@ -438,5 +438,5 @@
       <origin xyz="0 0 0" rpy="0 0 0"/>
       <geometry>
-    <box size="${camera_link} ${camera_link} ${camera_link}"/>
+    <box size="0.002 ${camera_link}  ${camera_link} "/>
       </geometry>
       <material name="red"/>

Commit message: fixed optical frame

File: elfin/elfin_description/urdf/elfin3.urdf_visualservo.xacro (robot description, xacro)
@@ -421,8 +421,8 @@
       link="elfin_end_link" />
   </joint>
+  <!-- NEW -->
   <joint name="camera_joint" type="fixed">
-    <axis xyz="0 0 0" />
-    <origin xyz="0 -0.079 0" rpy="${PI} 0 -${PI/2}"/>
-    <parent link="elfin_link6"/>
+    <origin xyz="0 0 -0.012" rpy="0 ${-PI/2} 0"/>
+    <parent link="elfin_end_link"/>
     <child link="camera_link"/>
   </joint>
@@ -432,5 +432,5 @@
       <origin xyz="0 0 0" rpy="0 0 0"/>
       <geometry>
-    <box size="${camera_link} ${camera_link} ${camera_link}"/>
+        <box size="0.002 ${camera_link} ${camera_link}"/>
       </geometry>
     </collision>
@@ -438,5 +438,5 @@
       <origin xyz="0 0 0" rpy="0 0 0"/>
       <geometry>
-    <box size="0.002 ${camera_link}  ${camera_link} "/>
+	<box size="0.002  ${camera_link} ${camera_link}"/>
       </geometry>
       <material name="red"/>
@@ -448,3 +448,14 @@
     </inertial>
   </link>
+  <!-- generate an optical frame http://www.ros.org/reps/rep-0103.html#suffix-frames
+      so that ros and opencv can operate on the camera frame correctly -->
+  <joint name="camera_optical_joint" type="fixed">
+    <!-- these values have to be these values otherwise the gazebo camera image
+        won't be aligned properly with the frame it is supposedly originating from -->
+    <origin xyz="0 0 0" rpy="${-PI/2} 0 ${-PI/2}"/>
+    <parent link="camera_link"/>
+    <child link="camera_link_optical"/>
+  </joint>
+  <link name="camera_link_optical">
+  </link>
 </robot>
